Commit message: Added the 'zed' to the simulation

File: src/sb_gazebo/urdf/jfrost.xacro (robot description, xacro)
@@ -19,5 +19,5 @@
 <xacro:property name="camera_size" value="0.05" />
 <xacro:property name="camera_mass" value="0.1" />
-<xacro:property name="camera_angle" value="0.5235" />
+<xacro:property name="camera_angle" value="${pi/8}" />
 <xacro:property name="lidar_size" value="0.05"/>
 <xacro:property name="lidar_elevation" value="0.1"/>
@@ -98,5 +98,5 @@
     <parent link="chassis"/>
     <child link="camera"/>
-    <origin xyz="${-(chassis_length/2) + camera_size} 0 ${chassis_height + chassis_elevation + tower_height + camera_size}" rpy="0 ${camera_angle} 0"/>
+    <origin xyz="${-(chassis_length/2)} 0 ${chassis_height + chassis_elevation + tower_height + camera_size}" rpy="0 ${camera_angle} 0"/>
 </joint>
 <link name="camera">

Commit message: Let there be ... proper orientation

File: src/sb_gazebo/urdf/jfrost.xacro (robot description, xacro)
@@ -120,4 +120,12 @@
   </inertial>
 </link>
+<!-- Hack to get the "zed" output to the right orientation -->
+<joint name="zed_orientation" type="fixed">
+    <parent link="camera"/>
+    <child link="zed_pointcloud"/>
+    <origin xyz="0 0 0" rpy="${-(pi/2)} 0 ${-(pi/2)}"/>
+</joint>
+<link name="zed_pointcloud" />
+<!-- End Hack -->
 <!-- Lidar -->
 <joint name="lidar_joint" type="fixed">

Commit message: Fixed gazebo xml files

File: src/sb_gazebo/urdf/jfrost.xacro (robot description, xacro)
@@ -75,5 +75,5 @@
         rpy="0 0 0"/>
   </joint>
-  <link name='tower_top_bar'>
+  <link name="tower_top_bar">
     <collision>
       <origin xyz="0 0 0" rpy="0 0 0"/>
